File: wiki/PCB.attach/gruvin9x-hacked.sch (KiCad schematic (older format))
At the start: 149 parts, among them P1 CONN_5X2, P2 CONN_5, P3 CONN_6, P4 CONN_9, P5 CONN_9, P6 CONN_6, P7 CONN_12, P8 CONN_30, Q1 2SC9014, SW1 SW_PUSH, SW2 SW_PUSH, SW3 SW_PUSH, SW4 SW_PUSH, SW5 SW_PUSH, SW6 SW_PUSH, U1 78L05, U2 4066, U3 LN-6206-30, X1 16MHz

Commit message: PDF and PS file updates
Parts:
- removed D?: DIODE, symbol DIODE
- removed JP?: JUMPER, symbol JUMPER
- removed K? (x2): CONN_3, symbol CONN_3
- removed Q?: NPN, symbol NPN
- removed R?: 33K, symbol R
- removed R? (x2): 10K, symbol R
- added D?: DIODE, symbol DIODE
- added PX: CONN_3, symbol CONN_3
- added Q?: NPN, symbol NPN
- added R68: 0, symbol R
- added R?: 33K, symbol R
- added R? (x2): 10K, symbol R
- gave numbers to parts that had none: 1
Connections:
- net labels added: FrSky_RXD, NC1_HACK, NC2_HACK, PC0_HACK, PG2_HACK
- wire segments 565 -> 468
- no-connect marks 10 -> 7
Other:
- note added: "HACK"
- note added: "INPUT: Fr-Sky RXD converted to TTL\nSIL3 hot-glued to main PCB\n"
- note added: "R17 removed"
- note added: "R7 removed"
- note added: "RS-232 +/12V"
- note added: "RS-232 to TTL inverter/level-shifter\nbuilt 'dead bug' style on spare space\nof the rear casing PCB."
- note added: "SPI Programming\nHeader"
- note removed: "RS-232 RXD"
- note removed: "SPI Programming Header"
- note removed: "TTL RXD"
- moved on the sheet: C10, C2, C22, C23, C24, C25, C26, C27, C28, C29, C3, C4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
