File: trunk/pcb/gruvin9x.sch (KiCad schematic (older format))
At the start: 151 parts, among them P1 CONN_5X2, P2 CONN_5, P3 CONN_6, P4 CONN_9, P5 CONN_9, P6 CONN_6, P7 CONN_12, P8 CONN_30, Q1 2SC9014, SW1 SW_PUSH, SW2 SW_PUSH, SW3 SW_PUSH, SW4 SW_PUSH, SW5 SW_PUSH, SW6 SW_PUSH, U1 78L05, U2 4066, U3 LN-6206-30, X1 16MHz

Commit message: PCB rev2.1 final_draft (gruvin9x.brd/sch) uploaded
Parts:
- removed D? (x14): DIODE, symbol DIODE
- removed R28, R29, R32: 200, symbol R
- added D10, D11, D12, D13, D14, D15, D2, D3, D4, D5, D6, D7, D8, D9: DIODESCH, symbol DIODESCH
- added P15: CONN_1, symbol CONN_1
- P13: renamed from P?; value CONN_7 -> CONN_8; symbol CONN_7 -> CONN_8
- gave numbers to parts that had none: 17
Connections:
- net labels added: Vcc_3V3
- net labels removed: SCK, SD_CLK
- wire segments 488 -> 484
Other:
- moved on the sheet: P10, R68
